File: input.kicad_sch (KiCad schematic)
At the start: 2 parts, among them J701 FCI10053363-200LF

Commit message: flesh out remote interface
Changed lines of the file:
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@@
     (stroke (width 0) (type solid) (color 0 0 0 0))
   )
-  (bus (pts (xy 140.97 144.78) (xy 101.6 144.78))
+  (bus (pts (xy 101.6 144.78) (xy 144.78 144.78))
     (stroke (width 0) (type solid) (color 0 0 0 0))
   )
@@
     (effects (font (size 1.27 1.27)) (justify right bottom))
   )
-  (label "{ps_interrupt ~present psok imonitor ~en}" (at 140.97 144.78 180)
-    (effects (font (size 1.27 1.27)) (justify right bottom))
-  )
   (label "~present" (at 142.24 123.19 0)
     (effects (font (size 1.27 1.27)) (justify left bottom))
   )
+  (label "{ps_interrupt ~present psok imonitor ~en}" (at 144.78 144.78 180)
+    (effects (font (size 1.27 1.27)) (justify right bottom))
+  )
   (label "ps_interrupt" (at 152.4 118.11 180)
