File: mpm3606.kicad_sch (KiCad schematic)
At the start: 6 parts, among them U1101 MPM3606

Commit message: flesh out remote interface
Parts:
- renumbered C1101 to C1201, C1102 to C1202, C1103 to C1203, FB1101 to FB1201, R1101 to R1201, U1101 to U1201
Changed lines of the file:
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@@
   (symbol (lib_id "proj_sym:Resistor") (at 111.76 50.8 0)
     (in_bom yes) (on_board yes)
-    (property "Reference" "R1101" (id 0) (at 113.03 50.1649 0)
+    (property "Reference" "R1201" (id 0) (at 113.03 50.1649 0)
       (effects (font (size 1.27 1.27)) (justify left))
     )
@@
   (symbol (lib_id "proj_sym:C_Polarized") (at 87.63 50.8 0)
     (in_bom yes) (on_board yes) (fields_autoplaced)
-    (property "Reference" "C1101" (id 0) (at 90.17 50.1649 0)
+    (property "Reference" "C1201" (id 0) (at 90.17 50.1649 0)
       (effects (font (size 1.27 1.27)) (justify left))
     )
@@
   (symbol (lib_id "proj_sym:C_Polarized") (at 168.91 50.8 0)
     (in_bom yes) (on_board yes) (fields_autoplaced)
-    (property "Reference" "C1103" (id 0) (at 171.45 50.1649 0)
+    (property "Reference" "C1203" (id 0) (at 171.45 50.1649 0)
       (effects (font (size 1.27 1.27)) (justify left))
     )
@@
   (symbol (lib_id "proj_sym:C") (at 100.33 50.8 0)
     (in_bom yes) (on_board yes)
-    (property "Reference" "C1102" (id 0) (at 102.87 50.1649 0)
+    (property "Reference" "C1202" (id 0) (at 102.87 50.1649 0)
       (effects (font (size 1.27 1.27)) (justify left))
     )
@@
   (symbol (lib_id "proj_sym:FerriteBead_Small") (at 83.82 48.26 90)
     (in_bom yes) (on_board yes) (fields_autoplaced)
-    (property "Reference" "FB1101" (id 0) (at 83.82 43.18 90))
+    (property "Reference" "FB1201" (id 0) (at 83.82 43.18 90))
     (property "Value" "100" (id 1) (at 83.82 45.72 90))
     (property "Footprint" "" (id 2) (at 83.82 50.038 90)
@@
   (symbol (lib_id "proj_sym:MPM3606") (at 132.08 71.12 0)
     (in_bom yes) (on_board yes) (fields_autoplaced)
-    (property "Reference" "U1101" (id 0) (at 131.445 34.29 0))
+    (property "Reference" "U1201" (id 0) (at 131.445 34.29 0))
     (property "Value" "MPM3606" (id 1) (at 131.445 36.83 0))
     (property "Footprint" "" (id 2) (at 132.08 71.12 0)
