File: mpm3811.kicad_sch (KiCad schematic)
At the start: 5 parts, among them U1001 MPM3811

Commit message: flesh out remote interface
Parts:
- renumbered C1001 to C1301, C1002 to C1302, C1003 to C1303, FB1001 to FB1301, U1001 to U1301
Changed lines of the file:
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@@
   (symbol (lib_id "power:PWR_FLAG") (at 125.73 93.98 0)
     (in_bom yes) (on_board yes) (fields_autoplaced)
-    (property "Reference" "#FLG01001" (id 0) (at 125.73 92.075 0)
+    (property "Reference" "#FLG01301" (id 0) (at 125.73 92.075 0)
       (effects (font (size 1.27 1.27)) hide)
     )
@@
   (symbol (lib_id "proj_sym:C_Polarized") (at 111.76 96.52 0)
     (in_bom yes) (on_board yes) (fields_autoplaced)
-    (property "Reference" "C1001" (id 0) (at 114.3 95.8849 0)
+    (property "Reference" "C1301" (id 0) (at 114.3 95.8849 0)
       (effects (font (size 1.27 1.27)) (justify left))
     )
@@
   (symbol (lib_id "proj_sym:C_Polarized") (at 163.83 96.52 0)
     (in_bom yes) (on_board yes) (fields_autoplaced)
-    (property "Reference" "C1003" (id 0) (at 166.37 95.8849 0)
+    (property "Reference" "C1303" (id 0) (at 166.37 95.8849 0)
       (effects (font (size 1.27 1.27)) (justify left))
     )
@@
   (symbol (lib_id "proj_sym:C") (at 121.92 96.52 0)
     (in_bom yes) (on_board yes) (fields_autoplaced)
-    (property "Reference" "C1002" (id 0) (at 124.46 95.8849 0)
+    (property "Reference" "C1302" (id 0) (at 124.46 95.8849 0)
       (effects (font (size 1.27 1.27)) (justify left))
     )
@@
   (symbol (lib_id "proj_sym:FerriteBead_Small") (at 107.95 93.98 90)
     (in_bom yes) (on_board yes) (fields_autoplaced)
-    (property "Reference" "FB1001" (id 0) (at 107.95 88.9 90))
+    (property "Reference" "FB1301" (id 0) (at 107.95 88.9 90))
     (property "Value" "100" (id 1) (at 107.95 91.44 90))
     (property "Footprint" "" (id 2) (at 107.95 95.758 90)
@@
   (symbol (lib_id "proj_sym:MPM3811") (at 140.97 104.14 0)
     (in_bom yes) (on_board yes) (fields_autoplaced)
-    (property "Reference" "U1001" (id 0) (at 140.97 88.9 0))
+    (property "Reference" "U1301" (id 0) (at 140.97 88.9 0))
     (property "Value" "MPM3811" (id 1) (at 140.97 91.44 0))
     (property "Footprint" "" (id 2) (at 140.97 104.14 0)
