File: output.kicad_sch (KiCad schematic)
At the start: 3 parts, among them J601 PCIe_8-Pin, J602 PCIe_8-Pin

Commit message: flesh out remote interface
Parts:
- gave numbers to parts that had none: 1
Changed lines of the file:
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@@
     (effects (font (size 1.27 1.27)) (justify left))
   )
-  (hierarchical_label "3.3V_{sense}" (shape input) (at 160.02 62.23 0)
+  (hierarchical_label "3.3V_{sense}" (shape output) (at 160.02 62.23 0)
     (effects (font (size 1.27 1.27)) (justify left))
   )
@@
   (symbol (lib_id "proj_sym:ATX-24") (at 143.51 57.15 0) (unit 1)
     (in_bom yes) (on_board yes) (fields_autoplaced)
-    (property "Reference" "J?" (id 0) (at 134.62 43.18 0))
+    (property "Reference" "J603" (id 0) (at 134.62 43.18 0))
     (property "Value" "ATX-24" (id 1) (at 149.86 43.18 0))
     (property "Footprint" "" (id 2) (at 143.51 59.69 0)
       (effects (font (size 1.27 1.27)) hide)
     )
-    (property "Datasheet" "${KIPRJMOD}/atx/power-supply-design-guide-june.pdf#page=33" (id 3) (at 204.47 71.12 0)
+    (property "Datasheet" "${KIPRJMOD}/atx/power-supply-design-guide-june.pdf" (id 3) (at 204.47 71.12 0)
       (effects (font (size 1.27 1.27)) hide)
     )
