File: control.kicad_sch (KiCad schematic)
At the start: 0 parts

Commit message: flesh out remote interface
Parts:
- added U? (x5): ICE40HX8K-BG121, Package_BGA:BGA-121_9.0x9.0mm_Layout11x11_P0.8mm_Ball0.4mm_Pad0.35mm_NSMD, symbol proj_sym:ICE40HX8K-BG121
Connections:
- new net: U?.D4 (VCC), U?.D8 (VCC), U?.H4 (VCC), U?.H8 (VCC)
- new net: U?.E5 (GND), U?.E6 (GND), U?.E7 (GND), U?.F5 (GND), U?.F6 (GND), U?.F7 (GND), U?.G5 (GND), U?.G6 (GND), U?.G7 (GND), U?.H5 (GND)
- new net: U?.E4 (VCCIO_3), U?.G4 (VCCIO_3)

Commit message: start control logic architecture
Parts:
- added R?: 20k, symbol proj_sym:Resistor
- added R?: 41k2, symbol proj_sym:Resistor
- added R?: 10k, symbol proj_sym:Resistor
- added R?: 11k5, symbol proj_sym:Resistor
- added RN201, RN202: 10k, symbol proj_sym:R_Pack04_Split
- added U202: TMUX1104, symbol proj_sym:TMUX1104
- added U203: SLG46621, symbol proj_sym:SLG46621
- gave numbers to parts that had none: 1
Connections:
- net 3.3V_{aux}: now also U203.14 (V_{dd2})
- net GND: now also R?.2, R?.2, RN201.2 (R2.1), RN201.4 (R4.1), RN202.2 (R2.1), U202.3 (GND)
- new net 3.3V_{divided}: RN201.3 (R3.1), RN201.5 (R4.2), U202.9 (S_{2})
- new net 3.3V_{th}: R?.1, R?.2
- new net 5V_{aux}: U202.6 (V_{dd}), U203.1 (V_{dd})
- new net 5V_{divided}: RN201.1 (R1.1), RN201.7 (R2.2), U202.2 (S_{1})
- new net 5V_{th}: R?.1, R?.2
- new net control_{cs}.imonitor: RN202.8 (R1.2)
- new net control_{cs}.psok: U202.4 (S_{3})
- new net control_{main}.3.3V: R?.1, RN201.6 (R3.2)
- new net control_{main}.5V: R?.1, RN201.8 (R1.2)
- new net imonitor_{divided}: RN202.1 (R1.1), RN202.7 (R2.2), U202.7 (S_{4})
- new net mux_{addr}.A_{0}: U202.1 (A_{0})
- new net mux_{addr}.A_{1}: U202.10 (A_{1})
- new net mux_{en}: U202.5 (EN)
- new net mux_{out}: U202.8 (D)
Other:
- note added: "3.00V"
- note added: "3.3V rail lower limit is"
- note added: "4.58V"
- note added: "5V rail lower limit is"
- note added: "V_{th} is nominally 1V at lower power rail tolerance limit."

Commit message: tweak schematic
Parts:
- removed U201: ICE40HX8K-BG121, Package_BGA:BGA-121_9.0x9.0mm_Layout11x11_P0.8mm_Ball0.4mm_Pad0.35mm_NSMD, symbol proj_sym:ICE40HX8K-BG121
- added R205: 20k, symbol proj_sym:Resistor
- added R206: 10k, symbol proj_sym:Resistor
- gave numbers to parts that had none: 4
- renumbered U202 to U201, U203 to U202
Connections:
- net GND: now also U202.11 (GND), R206.2
- net control_{cs}.psok: now also R205.1
- net mux_{out}: now also U202.8 (GPIO)
- net 3.3V_{divided} renamed 3.3V_{half}
- net 5V_{divided} renamed 5V_{half}
- net imonitor_{divided} renamed imonitor_{half}
- new net psok_{th}: R205.2, R206.1
- no-connect marks 0 -> 4
Other:
- added sheet FPGA (ice40hx8k.kicad_sch)
- note added: "control_{cs}.psok is nominally 3.3V for good power. psok_{th} will be >1V in this case."
- moved on the sheet: R201, R202, R203, R204, RN201A, RN201B, RN201C, RN201D, RN202A, RN202B, RN202C, RN202D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
