File: power.kicad_sch (KiCad schematic)
At the start: 15 parts

Commit message: flesh out remote interface
Parts:
- removed NT501, NT502: NetTie_2, symbol Device:NetTie_2
- added C501: 10u, symbol proj_sym:C_Polarized
- added FB501: 100, symbol proj_sym:FerriteBead_Small
- added Q501: Si2374DS, symbol proj_sym:Si2374DS
- added Q502, Q503: Si2333DDS, symbol proj_sym:Si2333DDS
- added R512: 100k, symbol proj_sym:Resistor
- added R515: 82k 1%, symbol proj_sym:Resistor
- added R516: 41k2 1%, symbol proj_sym:Resistor
- added R517: 10k, symbol proj_sym:Resistor
- R508: value 100k -> 10k
- renumbered R506 to R504, R507 to R505, R504 to R506, R505 to R507, R510 to R509, R511 to R510, R509 to R511, R512 to R513, R513 to R514
Connections:
- net 3.3V_{aux}: now also Q502.2 (S), R512.1, R517.1
- net GND: now also C501.2, Q501.2 (S), R516.2
- net ice_power.V_{core}: now also FB501.1
- net ice_power.V_{pll}: now also C501.1, FB501.2
- net ice_power.en: now also Q501.1 (G)
- new net: Q501.3 (D), Q502.1 (G), Q503.1 (G), R517.2
- new net 1.8V_{aux}: Q503.2 (S), R515.1
- new net MPM3811 Regulator 1.8V/FB: R515.2, R516.1
- new net MPM3811 Regulator 1.8V/en: R512.2
- new net ice_power.1.8V_{io}: Q503.3 (D)
- new net ice_power.3.3V_{io}: Q502.3 (D)
Other:
- sheet MPM3606 Regulator renamed MPM3606 3.3V
- sheet MPM3606 Regulator1 renamed MPM3606 5V
- sheet MPM3811 Regulator renamed MPM3811 1.2V
- sheet MPM3811 Regulator1 renamed MPM3811 Regulator 2.5V
- added sheet MPM3811 Regulator 1.8V (mpm3811.kicad_sch)
- note added: "FB voltage is nominally 0.6V; Recommended resistor values for 1.8V are 82k and 41.2k"
- moved on the sheet: R504, R505, R509, R510

Commit message: tweak schematic
Parts:
- Q501: value Si2374DS -> FDV301N; symbol proj_sym:Si2374DS -> proj_sym:FDV301N
Connections:
- net GND: now also Q501.S; no longer Q501.2 (S)
- net ice_power.en: now also Q501.G; no longer Q501.1 (G)
- net at Q502.1 (G), Q503.1 (G), R517.2: now also Q501.D; no longer Q501.3 (D)
Changed lines of the file:
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@@
     (pin "2")
   )
-  (symbol (lib_id "proj_sym:Si2374DS") (at 254 168.91 0) (unit 1)
+  (symbol (lib_id "proj_sym:FDV301N") (at 254 168.91 0) (unit 1)
     (in_bom yes) (on_board yes) (fields_autoplaced)
-    (property "Reference" "Q501" (id 0) (at 259.08 168.2749 0)
+    (property "Reference" "Q501" (id 0) (at 259.08 167.005 0)
       (effects (font (size 1.27 1.27)) (justify left))
     )
-    (property "Value" "Si2374DS" (id 1) (at 259.08 170.8149 0)
+    (property "Value" "FDV301N" (id 1) (at 259.08 168.91 0)
       (effects (font (size 1.27 1.27)) (justify left))
     )
@@
       (effects (font (size 1.27 1.27) italic) (justify left) hide)
     )
-    (property "Datasheet" "${KIPRJMOD}/si2374ds/si2374ds-1764268.pdf" (id 3) (at 254 168.91 0)
+    (property "Datasheet" "${KIPRJMOD}/fdv301n/FDV301N_D-2313106.pdf" (id 3) (at 254 168.91 0)
       (effects (font (size 1.27 1.27)) (justify left) hide)
     )
-    (pin "1")
-    (pin "2")
-    (pin "3")
+    (pin "D")
+    (pin "G")
+    (pin "S")
   )
   (symbol (lib_id "proj_sym:Si2333DDS") (at 256.54 147.32 270) (mirror x) (unit 1)
