File: remote.kicad_sch (KiCad schematic)
At the start: 25 parts, among them J301 GMJXHT-MM-S-88, T301 HX6062NL, U301 LTC2855, U302 LTC6820HMS, U303 LTC6820HMS

Commit message: start control logic architecture
Connections:
- net 3.3V_{AUX}: no longer C301.1, R301.1, R305.1, U301.12 (V_{cc}), U301.5 (TE), U302.1 (EN), U302.8 (PHA), U303.1 (EN), U303.12 (MSTR), U303.8 (PHA)
- new net 3.3V_{aux}: C301.1, R301.1, R305.1, U301.12 (V_{cc}), U301.5 (TE), U302.1 (EN), U302.8 (PHA), U303.1 (EN), U303.12 (MSTR), U303.8 (PHA)
Changed lines of the file:
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@@
     (effects (font (size 1.27 1.27)) (justify left bottom))
   )
-  (label "3.3V_{AUX}" (at 16.51 60.96 0)
-    (effects (font (size 1.27 1.27)) (justify left bottom))
-  )
-  (label "3.3V_{AUX}" (at 20.32 110.49 270)
+  (label "3.3V_{aux}" (at 16.51 60.96 0)
+    (effects (font (size 1.27 1.27)) (justify left bottom))
+  )
+  (label "3.3V_{aux}" (at 20.32 110.49 270)
     (effects (font (size 1.27 1.27)) (justify right bottom))
   )
@@
     (effects (font (size 1.27 1.27)) (justify left bottom))
   )
-  (label "3.3V_{AUX}" (at 44.45 50.8 0)
+  (label "3.3V_{aux}" (at 44.45 50.8 0)
     (effects (font (size 1.27 1.27)) (justify left bottom))
   )
@@
     (effects (font (size 1.27 1.27)) (justify right bottom))
   )
-  (label "phantom_power" (at 54.61 27.94 180)
-    (effects (font (size 1.27 1.27)) (justify right bottom))
-  )
-  (label "GND" (at 54.61 30.48 180)
-    (effects (font (size 1.27 1.27)) (justify right bottom))
-  )
-  (label "3.3V_{AUX}" (at 54.61 33.02 180)
-    (effects (font (size 1.27 1.27)) (justify right bottom))
-  )
   (label "GND" (at 59.69 60.96 90)
     (effects (font (size 1.27 1.27)) (justify left bottom))
@@
     (effects (font (size 1.27 1.27)) (justify left bottom))
   )
-  (label "3.3V_{AUX}" (at 87.63 102.87 180)
+  (label "3.3V_{aux}" (at 87.63 102.87 180)
     (effects (font (size 1.27 1.27)) (justify right bottom))
   )
@@
     (effects (font (size 1.27 1.27)) (justify right bottom))
   )
-  (label "3.3V_{AUX}" (at 152.4 107.95 270)
+  (label "3.3V_{aux}" (at 152.4 107.95 270)
     (effects (font (size 1.27 1.27)) (justify right bottom))
   )
@@
     (effects (font (size 1.27 1.27)) (justify left bottom))
   )
-  (label "3.3V_{AUX}" (at 213.36 102.87 180)
+  (label "3.3V_{aux}" (at 213.36 102.87 180)
     (effects (font (size 1.27 1.27)) (justify right bottom))
   )
@@
     (effects (font (size 1.27 1.27)) (justify right))
   )
-  (hierarchical_label "3.3V_{AUX}" (shape input) (at 39.37 33.02 180)
+  (hierarchical_label "3.3V_{aux}" (shape input) (at 39.37 33.02 180)
     (effects (font (size 1.27 1.27)) (justify right))
   )

Commit message: tweak schematic
Connections:
- net 3.3V_{AUX} is gone; now on net 3.3V_{aux}: C304.1, C306.1, U302.6 (VddS), U302.9 (Vdd), U303.6 (VddS), U303.9 (Vdd)
- net 3.3V_{aux}: now also U302.7 (POL), U303.7 (POL)
- net GND: no longer U302.7 (POL), U303.7 (POL)
Other:
- note added: "iCE40 configuration hardware latches data on SCK rising edge."
Changed lines of the file:
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@@
   (junction (at 27.94 105.41) (diameter 0.9144) (color 0 0 0 0))
   (junction (at 76.2 102.87) (diameter 0.9144) (color 0 0 0 0))
-  (junction (at 76.2 110.49) (diameter 0.9144) (color 0 0 0 0))
-  (junction (at 76.2 113.03) (diameter 0.9144) (color 0 0 0 0))
   (junction (at 76.2 132.08) (diameter 0.9144) (color 0 0 0 0))
+  (junction (at 78.74 113.03) (diameter 0.9144) (color 0 0 0 0))
+  (junction (at 81.28 102.87) (diameter 0.9144) (color 0 0 0 0))
   (junction (at 85.09 165.1) (diameter 0.9144) (color 0 0 0 0))
   (junction (at 87.63 120.65) (diameter 0.9144) (color 0 0 0 0))
@@
   (junction (at 201.93 102.87) (diameter 0.9144) (color 0 0 0 0))
   (junction (at 201.93 105.41) (diameter 0.9144) (color 0 0 0 0))
-  (junction (at 201.93 113.03) (diameter 0.9144) (color 0 0 0 0))
+  (junction (at 201.93 107.95) (diameter 0.9144) (color 0 0 0 0))
   (junction (at 201.93 132.08) (diameter 0.9144) (color 0 0 0 0))
   (junction (at 213.36 62.23) (diameter 0.9144) (color 0 0 0 0))
@@
     (stroke (width 0) (type solid) (color 0 0 0 0))
   )
-  (wire (pts (xy 76.2 102.87) (xy 87.63 102.87))
-    (stroke (width 0) (type solid) (color 0 0 0 0))
-  )
-  (wire (pts (xy 76.2 107.95) (xy 76.2 110.49))
-    (stroke (width 0) (type solid) (color 0 0 0 0))
-  )
-  (wire (pts (xy 76.2 110.49) (xy 76.2 113.03))
-    (stroke (width 0) (type solid) (color 0 0 0 0))
-  )
-  (wire (pts (xy 76.2 113.03) (xy 87.63 113.03))
+  (wire (pts (xy 76.2 102.87) (xy 81.28 102.87))
+    (stroke (width 0) (type solid) (color 0 0 0 0))
+  )
+  (wire (pts (xy 76.2 107.95) (xy 78.74 107.95))
+    (stroke (width 0) (type solid) (color 0 0 0 0))
+  )
+  (wire (pts (xy 76.2 110.49) (xy 81.28 110.49))
+    (stroke (width 0) (type solid) (color 0 0 0 0))
+  )
+  (wire (pts (xy 76.2 113.03) (xy 78.74 113.03))
     (stroke (width 0) (type solid) (color 0 0 0 0))
   )
@@
     (stroke (width 0) (type solid) (color 0 0 0 0))
   )
+  (wire (pts (xy 78.74 107.95) (xy 78.74 113.03))
+    (stroke (width 0) (type solid) (color 0 0 0 0))
+  )
+  (wire (pts (xy 78.74 113.03) (xy 87.63 113.03))
+    (stroke (width 0) (type solid) (color 0 0 0 0))
+  )
   (wire (pts (xy 78.74 165.1) (xy 85.09 165.1))
     (stroke (width 0) (type solid) (color 0 0 0 0))
@@
     (stroke (width 0) (type solid) (color 0 0 0 0))
   )
+  (wire (pts (xy 81.28 102.87) (xy 87.63 102.87))
+    (stroke (width 0) (type solid) (color 0 0 0 0))
+  )
+  (wire (pts (xy 81.28 110.49) (xy 81.28 102.87))
+    (stroke (width 0) (type solid) (color 0 0 0 0))
+  )
   (wire (pts (xy 85.09 137.16) (xy 85.09 140.97))
     (stroke (width 0) (type solid) (color 0 0 0 0))
@@
     (stroke (width 0) (type solid) (color 0 0 0 0))
   )
-  (wire (pts (xy 201.93 110.49) (xy 201.93 113.03))
+  (wire (pts (xy 201.93 107.95) (xy 201.93 110.49))
     (stroke (width 0) (type solid) (color 0 0 0 0))
   )
@@
     (stroke (width 0) (type solid) (color 0 0 0 0))
   )
+  (text "iCE40 configuration hardware latches data on SCK rising edge."
+    (at 27.94 93.98 0)
+    (effects (font (size 1.27 1.27)) (justify left bottom))
+  )
   (label "DSER.RX" (at 16.51 50.8 0)
     (effects (font (size 1.27 1.27)) (justify left bottom))
@@
     (effects (font (size 1.27 1.27)) (justify right bottom))
   )
-  (label "3.3V_{AUX}" (at 85.09 132.08 180)
+  (label "3.3V_{aux}" (at 85.09 132.08 180)
     (effects (font (size 1.27 1.27)) (justify right bottom))
   )
@@
     (effects (font (size 1.27 1.27)) (justify right bottom))
   )
-  (label "3.3V_{AUX}" (at 210.82 132.08 180)
-    (effects (font (size 1.27 1.27)) (justify right bottom))
-  )
+  (label "3.3V_{aux}" (at 210.82 132.08 180)
+    (effects (font (size 1.27 1.27)) (justify right bottom))
+  )
